File: Hardware/Tiny_Programmer.sch (EAGLE design)
At the start: 31 parts, among them Q1 16MHz, U1 ATTINY84, X1 USB-A-H

Commit message: Revert "Modifies the new 6-pin SIP to be more compatible with an FTDI."
This reverts commit e9ce5eee6c851359ce4a9d7fdec24ce809564be4.
Parts:
- removed JP12: (no value), SparkFun-Connectors:M06SIP
- added JP10: (no value), SparkFun-Connectors:M06SIP
Connections:
- net GND: now also JP10.5; no longer JP12.6
- net MISO: now also JP10.3; no longer JP12.3
- net MOSI: now also JP10.4; no longer JP12.2
- net RST: now also JP10.1; no longer JP12.1
- net SCK: now also JP10.2; no longer JP12.5
- net VCC: now also JP10.6; no longer JP12.4
Changed lines of the file:
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@@
 <?xml version="1.0" encoding="utf-8"?>
 <!DOCTYPE eagle SYSTEM "eagle.dtd">
-<eagle version="6.5.0">
+<eagle version="6.4">
 <drawing>
 <settings>
@@
 <layer number="106" name="bPlate" color="7" fill="1" visible="yes" active="yes"/>
 <layer number="107" name="Crop" color="7" fill="1" visible="yes" active="yes"/>
-<layer number="108" name="tplace-old" color="10" fill="1" visible="yes" active="yes"/>
-<layer number="109" name="ref-old" color="11" fill="1" visible="yes" active="yes"/>
 <layer number="116" name="Patch_BOT" color="9" fill="4" visible="yes" active="yes"/>
 <layer number="121" name="_tsilk" color="7" fill="1" visible="yes" active="yes"/>
@@
 <part name="GND17" library="SparkFun-Aesthetics" deviceset="GND" device=""/>
 <part name="GND18" library="SparkFun-Aesthetics" deviceset="GND" device=""/>
+<part name="JP10" library="SparkFun-Connectors" deviceset="M06" device="SIP"/>
+<part name="GND1" library="SparkFun-Aesthetics" deviceset="GND" device=""/>
+<part name="SUPPLY9" library="SparkFun-Aesthetics" deviceset="VCC" device=""/>
 <part name="JP11" library="SparkFun-Aesthetics" deviceset="LOGO-SFE" device="SK"/>
-<part name="JP12" library="SparkFun-Connectors" deviceset="M06" device="SIP"/>
-<part name="P+4" library="SparkFun" deviceset="VCC" device=""/>
-<part name="GND2" library="SparkFun" deviceset="GND" device=""/>
 </parts>
 <sheets>
@@
 <instance part="GND17" gate="1" x="20.32" y="30.48"/>
 <instance part="GND18" gate="1" x="40.64" y="30.48"/>
+<instance part="JP10" gate="G$1" x="111.76" y="38.1"/>
+<instance part="GND1" gate="1" x="119.38" y="27.94"/>
+<instance part="SUPPLY9" gate="1" x="119.38" y="48.26"/>
 <instance part="JP11" gate="G$1" x="241.3" y="38.1"/>
-<instance part="JP12" gate="G$1" x="116.84" y="38.1"/>
-<instance part="P+4" gate="1" x="127" y="48.26"/>
-<instance part="GND2" gate="1" x="124.46" y="25.4"/>
 </instances>
 <busses>
@@
 </segment>
 <segment>
-<pinref part="JP12" gate="G$1" pin="4"/>
-<pinref part="P+4" gate="1" pin="VCC"/>
-<wire x1="121.92" y1="40.64" x2="127" y2="40.64" width="0.1524" layer="91"/>
-<wire x1="127" y1="40.64" x2="127" y2="48.26" width="0.1524" layer="91"/>
+<pinref part="JP10" gate="G$1" pin="6"/>
+<wire x1="116.84" y1="45.72" x2="119.38" y2="45.72" width="0.1524" layer="91"/>
+<wire x1="119.38" y1="45.72" x2="119.38" y2="48.26" width="0.1524" layer="91"/>
+<pinref part="SUPPLY9" gate="1" pin="VCC"/>
 </segment>
 </net>
@@
 </segment>
 <segment>
-<wire x1="124.46" y1="45.72" x2="124.46" y2="27.94" width="0.1524" layer="91"/>
-<pinref part="GND2" gate="1" pin="GND"/>
-<pinref part="JP12" gate="G$1" pin="6"/>
-<wire x1="121.92" y1="45.72" x2="124.46" y2="45.72" width="0.1524" layer="91"/>
+<pinref part="JP10" gate="G$1" pin="5"/>
+<wire x1="116.84" y1="43.18" x2="119.38" y2="43.18" width="0.1524" layer="91"/>
+<wire x1="119.38" y1="43.18" x2="119.38" y2="30.48" width="0.1524" layer="91"/>
+<pinref part="GND1" gate="1" pin="GND"/>
 </segment>
 </net>
@@
 </segment>
 <segment>
-<pinref part="JP12" gate="G$1" pin="2"/>
-<wire x1="121.92" y1="35.56" x2="129.54" y2="35.56" width="0.1524" layer="91"/>
-<label x="129.54" y="35.56" size="1.27" layer="95" xref="yes"/>
+<label x="124.46" y="40.64" size="1.27" layer="95" xref="yes"/>
+<pinref part="JP10" gate="G$1" pin="4"/>
+<wire x1="116.84" y1="40.64" x2="124.46" y2="40.64" width="0.1524" layer="91"/>
 </segment>
 </net>
@@
 </segment>
 <segment>
-<pinref part="JP12" gate="G$1" pin="3"/>
-<wire x1="121.92" y1="38.1" x2="129.54" y2="38.1" width="0.1524" layer="91"/>
-<label x="129.54" y="38.1" size="1.27" layer="95" xref="yes"/>
+<label x="124.46" y="38.1" size="1.27" layer="95" xref="yes"/>
+<pinref part="JP10" gate="G$1" pin="3"/>
+<wire x1="116.84" y1="38.1" x2="124.46" y2="38.1" width="0.1524" layer="91"/>
 </segment>
 </net>
@@
 </segment>
 <segment>
-<pinref part="JP12" gate="G$1" pin="5"/>
-<wire x1="121.92" y1="43.18" x2="129.54" y2="43.18" width="0.1524" layer="91"/>
-<label x="129.54" y="43.18" size="1.27" layer="95" xref="yes"/>
+<label x="124.46" y="35.56" size="1.27" layer="95" xref="yes"/>
+<pinref part="JP10" gate="G$1" pin="2"/>
+<wire x1="116.84" y1="35.56" x2="124.46" y2="35.56" width="0.1524" layer="91"/>
 </segment>
 </net>
@@
 </segment>
 <segment>
-<pinref part="JP12" gate="G$1" pin="1"/>
-<wire x1="121.92" y1="33.02" x2="129.54" y2="33.02" width="0.1524" layer="91"/>
-<label x="129.54" y="33.02" size="1.27" layer="95" xref="yes"/>
-</segment>
-</net>
+<label x="124.46" y="33.02" size="1.27" layer="95" xref="yes"/>
+<pinref part="JP10" gate="G$1" pin="1"/>
+<wire x1="124.46" y1="33.02" x2="116.84" y2="33.02" width="0.1524" layer="91"/>
+</segment>
+</net>

Commit message: Modifies the new 6-pin SIP to be more compatible with an FTDI.
The new pin out should allow MOSI and MISO to bit-bang serial and
communicate over an FTDI connection for serial debuggin.
Parts:
- removed JP10: (no value), SparkFun-Connectors:M06SIP
- added JP12: (no value), SparkFun-Connectors:M06SIP
Connections:
- net GND: now also JP12.6; no longer JP10.5
- net MISO: now also JP12.3; no longer JP10.3
- net MOSI: now also JP12.2; no longer JP10.4
- net RST: now also JP12.1; no longer JP10.1
- net SCK: now also JP12.5; no longer JP10.2
- net VCC: now also JP12.4; no longer JP10.6
Changed lines of the file:
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@@
 <?xml version="1.0" encoding="utf-8"?>
 <!DOCTYPE eagle SYSTEM "eagle.dtd">
-<eagle version="6.4">
+<eagle version="6.5.0">
 <drawing>
 <settings>
@@
 <layer number="106" name="bPlate" color="7" fill="1" visible="yes" active="yes"/>
 <layer number="107" name="Crop" color="7" fill="1" visible="yes" active="yes"/>
+<layer number="108" name="tplace-old" color="10" fill="1" visible="yes" active="yes"/>
+<layer number="109" name="ref-old" color="11" fill="1" visible="yes" active="yes"/>
 <layer number="116" name="Patch_BOT" color="9" fill="4" visible="yes" active="yes"/>
 <layer number="121" name="_tsilk" color="7" fill="1" visible="yes" active="yes"/>
@@
 <part name="GND17" library="SparkFun-Aesthetics" deviceset="GND" device=""/>
 <part name="GND18" library="SparkFun-Aesthetics" deviceset="GND" device=""/>
-<part name="JP10" library="SparkFun-Connectors" deviceset="M06" device="SIP"/>
-<part name="GND1" library="SparkFun-Aesthetics" deviceset="GND" device=""/>
-<part name="SUPPLY9" library="SparkFun-Aesthetics" deviceset="VCC" device=""/>
 <part name="JP11" library="SparkFun-Aesthetics" deviceset="LOGO-SFE" device="SK"/>
+<part name="JP12" library="SparkFun-Connectors" deviceset="M06" device="SIP"/>
+<part name="P+4" library="SparkFun" deviceset="VCC" device=""/>
+<part name="GND2" library="SparkFun" deviceset="GND" device=""/>
 </parts>
 <sheets>
@@
 <instance part="GND17" gate="1" x="20.32" y="30.48"/>
 <instance part="GND18" gate="1" x="40.64" y="30.48"/>
-<instance part="JP10" gate="G$1" x="111.76" y="38.1"/>
-<instance part="GND1" gate="1" x="119.38" y="27.94"/>
-<instance part="SUPPLY9" gate="1" x="119.38" y="48.26"/>
 <instance part="JP11" gate="G$1" x="241.3" y="38.1"/>
+<instance part="JP12" gate="G$1" x="116.84" y="38.1"/>
+<instance part="P+4" gate="1" x="127" y="48.26"/>
+<instance part="GND2" gate="1" x="124.46" y="25.4"/>
 </instances>
 <busses>
@@
 </segment>
 <segment>
-<pinref part="JP10" gate="G$1" pin="6"/>
-<wire x1="116.84" y1="45.72" x2="119.38" y2="45.72" width="0.1524" layer="91"/>
-<wire x1="119.38" y1="45.72" x2="119.38" y2="48.26" width="0.1524" layer="91"/>
-<pinref part="SUPPLY9" gate="1" pin="VCC"/>
+<pinref part="JP12" gate="G$1" pin="4"/>
+<pinref part="P+4" gate="1" pin="VCC"/>
+<wire x1="121.92" y1="40.64" x2="127" y2="40.64" width="0.1524" layer="91"/>
+<wire x1="127" y1="40.64" x2="127" y2="48.26" width="0.1524" layer="91"/>
 </segment>
 </net>
@@
 </segment>
 <segment>
-<pinref part="JP10" gate="G$1" pin="5"/>
-<wire x1="116.84" y1="43.18" x2="119.38" y2="43.18" width="0.1524" layer="91"/>
-<wire x1="119.38" y1="43.18" x2="119.38" y2="30.48" width="0.1524" layer="91"/>
-<pinref part="GND1" gate="1" pin="GND"/>
+<wire x1="124.46" y1="45.72" x2="124.46" y2="27.94" width="0.1524" layer="91"/>
+<pinref part="GND2" gate="1" pin="GND"/>
+<pinref part="JP12" gate="G$1" pin="6"/>
+<wire x1="121.92" y1="45.72" x2="124.46" y2="45.72" width="0.1524" layer="91"/>
 </segment>
 </net>
@@
 </segment>
 <segment>
-<label x="124.46" y="40.64" size="1.27" layer="95" xref="yes"/>
-<pinref part="JP10" gate="G$1" pin="4"/>
-<wire x1="116.84" y1="40.64" x2="124.46" y2="40.64" width="0.1524" layer="91"/>
+<pinref part="JP12" gate="G$1" pin="2"/>
+<wire x1="121.92" y1="35.56" x2="129.54" y2="35.56" width="0.1524" layer="91"/>
+<label x="129.54" y="35.56" size="1.27" layer="95" xref="yes"/>
 </segment>
 </net>
@@
 </segment>
 <segment>
-<label x="124.46" y="38.1" size="1.27" layer="95" xref="yes"/>
-<pinref part="JP10" gate="G$1" pin="3"/>
-<wire x1="116.84" y1="38.1" x2="124.46" y2="38.1" width="0.1524" layer="91"/>
+<pinref part="JP12" gate="G$1" pin="3"/>
+<wire x1="121.92" y1="38.1" x2="129.54" y2="38.1" width="0.1524" layer="91"/>
+<label x="129.54" y="38.1" size="1.27" layer="95" xref="yes"/>
 </segment>
 </net>
@@
 </segment>
 <segment>
-<label x="124.46" y="35.56" size="1.27" layer="95" xref="yes"/>
-<pinref part="JP10" gate="G$1" pin="2"/>
-<wire x1="116.84" y1="35.56" x2="124.46" y2="35.56" width="0.1524" layer="91"/>
+<pinref part="JP12" gate="G$1" pin="5"/>
+<wire x1="121.92" y1="43.18" x2="129.54" y2="43.18" width="0.1524" layer="91"/>
+<label x="129.54" y="43.18" size="1.27" layer="95" xref="yes"/>
 </segment>
 </net>
@@
 </segment>
 <segment>
-<label x="124.46" y="33.02" size="1.27" layer="95" xref="yes"/>
-<pinref part="JP10" gate="G$1" pin="1"/>
-<wire x1="124.46" y1="33.02" x2="116.84" y2="33.02" width="0.1524" layer="91"/>
-</segment>
-</net>
+<pinref part="JP12" gate="G$1" pin="1"/>
+<wire x1="121.92" y1="33.02" x2="129.54" y2="33.02" width="0.1524" layer="91"/>
+<label x="129.54" y="33.02" size="1.27" layer="95" xref="yes"/>
+</segment>
+</net>

Commit message: Adding version number to schematic
Other:
- note added: "v13"
Changed lines of the file:
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@@
 <?xml version="1.0" encoding="utf-8"?>
 <!DOCTYPE eagle SYSTEM "eagle.dtd">
-<eagle version="6.5.0">
+<eagle version="7.4.0">
 <drawing>
 <settings>
@@
 <layer number="254" name="cooling" color="7" fill="1" visible="yes" active="yes"/>
 </layers>
-<schematic>
+<schematic xreflabel="%F%N/%S" xrefpart="/%S">
 <attributes>
 </attributes>
@@
 <text x="198.12" y="172.72" size="1.778" layer="97">Added 6-pin SIP to end of board</text>
 <text x="198.12" y="170.18" size="1.778" layer="97">Added comments to schematic</text>
+<text x="241.3" y="7.62" size="1.27" layer="94">v13</text>
 </plain>
 <instances>
